Commit message: kuka shelf experiment now training ready mostly

File: world/obstacles/shelf/shelf.urdf (robot description, URDF)
Before this commit: robot maze, 61 links, 60 joints
Links:
- removed link link_40
- removed link link_41
- removed link link_42
- removed link link_43
- removed link link_44
- removed link link_45
- removed link link_46
- removed link link_47
- removed link link_48
- removed link link_49
- removed link link_50
- removed link link_51
- removed link link_52
- removed link link_53
- removed link link_54
- removed link link_55
- removed link link_56
- removed link link_57
- removed link link_58
- removed link link_59
- link link_0: geometry collision box size=0.36 0.01 0.5; visual box size=0.36 0.01 0.5
- link link_1: geometry collision box size=0.01 0.36 0.5; visual box size=0.01 0.36 0.5
- link link_10: geometry collision box size=0.01 0.36 0.5; visual box size=0.01 0.36 0.5
- link link_11: geometry collision box size=0.36 0.01 0.5; visual box size=0.36 0.01 0.5
- link link_12: geometry collision box size=0.01 0.36 0.5; visual box size=0.01 0.36 0.5
- link link_13: geometry collision box size=0.36 0.01 0.5; visual box size=0.36 0.01 0.5
- link link_14: geometry collision box size=0.01 0.36 0.5; visual box size=0.01 0.36 0.5
- link link_15: geometry collision box size=0.36 0.01 0.5; visual box size=0.36 0.01 0.5
- link link_16: geometry collision box size=0.01 0.36 0.5; visual box size=0.01 0.36 0.5
- link link_17: geometry collision box size=0.01 0.36 0.5; visual box size=0.01 0.36 0.5
- link link_18: geometry collision box size=0.36 0.01 0.5; visual box size=0.36 0.01 0.5
- link link_19: geometry collision box size=0.01 0.36 0.5; visual box size=0.01 0.36 0.5
- link link_2: geometry collision box size=0.36 0.01 0.5; visual box size=0.36 0.01 0.5
- link link_20: geometry collision box size=0.36 0.01 0.5; visual box size=0.36 0.01 0.5
- link link_21: geometry collision box size=0.01 0.36 0.5; visual box size=0.01 0.36 0.5
- link link_22: geometry collision box size=0.36 0.01 0.5; visual box size=0.36 0.01 0.5
- link link_23: geometry collision box size=0.01 0.36 0.5; visual box size=0.01 0.36 0.5
- link link_24: geometry collision box size=0.36 0.01 0.5; visual box size=0.36 0.01 0.5
- link link_25: geometry collision box size=0.01 0.36 0.5; visual box size=0.01 0.36 0.5
- link link_26: geometry collision box size=0.01 0.36 0.5; visual box size=0.01 0.36 0.5
- link link_27: geometry collision box size=0.36 0.01 0.5; visual box size=0.36 0.01 0.5
- link link_28: geometry collision box size=0.01 0.36 0.5; visual box size=0.01 0.36 0.5
- link link_29: geometry collision box size=0.36 0.01 0.5; visual box size=0.36 0.01 0.5
- link link_3: geometry collision box size=0.01 0.36 0.5; visual box size=0.01 0.36 0.5
- link link_30: geometry collision box size=0.36 0.01 0.5; visual box size=0.36 0.01 0.5
- link link_31: geometry collision box size=0.01 0.36 0.5; visual box size=0.01 0.36 0.5
- link link_32: geometry collision box size=0.36 0.01 0.5; visual box size=0.36 0.01 0.5
- link link_33: geometry collision box size=0.36 0.01 0.5; visual box size=0.36 0.01 0.5
- link link_34: geometry collision box size=0.01 0.36 0.5; visual box size=0.01 0.36 0.5
- link link_35: geometry collision box size=0.36 0.01 0.5; visual box size=0.36 0.01 0.5
- link link_36: geometry collision box size=0.36 0.01 0.5; visual box size=0.36 0.01 0.5
- link link_37: geometry collision box size=0.01 0.36 0.5; visual box size=0.01 0.36 0.5
- link link_38: geometry collision box size=0.01 0.36 0.5; visual box size=0.01 0.36 0.5
- link link_39: geometry collision box size=0.36 0.01 0.5; visual box size=0.36 0.01 0.5
- link link_4: geometry collision box size=0.36 0.01 0.5; visual box size=0.36 0.01 0.5
- link link_5: geometry collision box size=0.01 0.36 0.5; visual box size=0.01 0.36 0.5
- link link_6: geometry collision box size=0.36 0.01 0.5; visual box size=0.36 0.01 0.5
- link link_7: geometry collision box size=0.01 0.36 0.5; visual box size=0.01 0.36 0.5
- link link_8: geometry collision box size=0.01 0.36 0.5; visual box size=0.01 0.36 0.5
- link link_9: geometry collision box size=0.36 0.01 0.5; visual box size=0.36 0.01 0.5
Joints:
- removed joint joint_40
- removed joint joint_41
- removed joint joint_42
- removed joint joint_43
- removed joint joint_44
- removed joint joint_45
- removed joint joint_46
- removed joint joint_47
- removed joint joint_48
- removed joint joint_49
- removed joint joint_50
- removed joint joint_51
- removed joint joint_52
- removed joint joint_53
- removed joint joint_54
- removed joint joint_55
- removed joint joint_56
- removed joint joint_57
- removed joint joint_58
- removed joint joint_59
