Commit message: first integration of blender recorder

File: assets/robots/predefined/kr16/urdf/kr16.urdf (robot description, URDF)
Before this commit: robot kuka_kr16_2, 8 links, 7 joints
Links:
- link base_link: geometry collision mesh filename=../meshes/collision/base_link.stl; visual mesh filename=../meshes/visual/base_link.dae
- link link_1: geometry collision mesh filename=../meshes/collision/link_1.stl; visual mesh filename=../meshes/visual/link_1.dae
- link link_2: geometry collision mesh filename=../meshes/collision/link_2.stl; visual mesh filename=../meshes/visual/link_2.dae
- link link_3: geometry collision mesh filename=../meshes/collision/link_3.stl; visual mesh filename=../meshes/visual/link_3.dae
- link link_4: geometry collision mesh filename=../meshes/collision/link_4.stl; visual mesh filename=../meshes/visual/link_4.dae
- link link_5: geometry collision mesh filename=../meshes/collision/link_5.stl; visual mesh filename=../meshes/visual/link_5.dae
- link link_6: geometry collision mesh filename=../meshes/collision/link_6.stl; visual mesh filename=../meshes/visual/link_6.dae
