Commit message: updated ur5 joint limits

File: modular_drl_env/assets/robots/predefined/ur5/urdf/ur5.urdf (robot description, URDF)
Before this commit: robot ur5_with_torch, 9 links, 8 joints
Joints:
- joint elbow_joint: limit lower=-3.14159265359 upper=3.14159265359 effort=300.0 velocity=10 -> lower=-6.28318530718 upper=6.28318530718 effort=300.0 velocity=10
- joint shoulder_lift_joint: limit lower=-3.14159265359 upper=3.14159265359 effort=300.0 velocity=10 -> lower=-6.28318530718 upper=6.28318530718 effort=300.0 velocity=10
- joint shoulder_pan_joint: limit lower=-3.14159265359 upper=3.14159265359 effort=300.0 velocity=10 -> lower=-6.28318530718 upper=6.28318530718 effort=300.0 velocity=10
- joint wrist_1_joint: limit lower=-3.14159265359 upper=3.14159265359 effort=300.0 velocity=10 -> lower=-6.28318530718 upper=6.28318530718 effort=300.0 velocity=10
- joint wrist_2_joint: limit lower=-3.14159265359 upper=3.14159265359 effort=300.0 velocity=10 -> lower=-6.28318530718 upper=6.28318530718 effort=300.0 velocity=10
- joint wrist_3_joint: limit lower=-3.14159265359 upper=3.14159265359 effort=300.0 velocity=10 -> lower=-6.28318530718 upper=6.28318530718 effort=300.0 velocity=10

Commit message: small updates everywhere

File: modular_drl_env/assets/robots/predefined/ur5/urdf/ur5.urdf (robot description, URDF)
Before this commit: robot ur5_with_torch, 9 links, 8 joints
Joints:
- joint elbow_joint: limit lower=-6.28318530718 upper=6.28318530718 effort=300.0 velocity=10 -> lower=-3.14159265359 upper=3.14159265359 effort=300.0 velocity=10
- joint shoulder_lift_joint: limit lower=-6.28318530718 upper=6.28318530718 effort=300.0 velocity=10 -> lower=-3.14159265359 upper=3.14159265359 effort=300.0 velocity=10
- joint shoulder_pan_joint: limit lower=-6.28318530718 upper=6.28318530718 effort=300.0 velocity=10 -> lower=-3.14159265359 upper=3.14159265359 effort=300.0 velocity=10
- joint wrist_1_joint: limit lower=-6.28318530718 upper=6.28318530718 effort=300.0 velocity=10 -> lower=-3.14159265359 upper=3.14159265359 effort=300.0 velocity=10
- joint wrist_2_joint: limit lower=-6.28318530718 upper=6.28318530718 effort=300.0 velocity=10 -> lower=-3.14159265359 upper=3.14159265359 effort=300.0 velocity=10
- joint wrist_3_joint: limit lower=-6.28318530718 upper=6.28318530718 effort=300.0 velocity=10 -> lower=-3.14159265359 upper=3.14159265359 effort=300.0 velocity=10
